File: pcb/pcb.kicad_sch (KiCad schematic)
At the start: 0 parts

Commit message: documentation
Parts:
- added D1, D2, D3, D4, D5, D6, D7, D8, D9: D, symbol Device:D
- added D12, D13: SK6812MINI-E, SK6812MINI-E - 3.2x2.8x1.78mm, symbol SK6812MINI-E:SK6812MINI-E
- added J1: OLED_0.91_SSD1306, symbol Connector_Generic:Conn_01x04
- added SW1, SW2, SW3, SW4, SW5, SW6, SW7, SW8, SW9: SW_Push_45deg, symbol Switch:SW_Push_45deg
- added SW1: RotaryEncoder_Switch, symbol Device:RotaryEncoder_Switch
- added U1: MOUDLE-SEEEDUINO-XIAO, symbol XIAO_RP2040:MOUDLE-SEEEDUINO-XIAO
Connections:
- new net: D6.2 (A), SW6.2
- new net: D7.2 (A), SW7.2
- new net: D12.2 (DOUT), D13.4 (DIN)
- new net: D3.2 (A), SW3.2
- new net: D5.2 (A), SW5.2
- new net: D2.2 (A), SW2.2
- new net: D9.2 (A), SW9.2
- new net: D4.2 (A), SW4.2
- new net: D8.2 (A), SW8.2
- new net: D1.2 (A), SW1.2
- new net +3V3: U1.12 (3V3)
- new net +5V: D12.1 (VDD), D13.1 (VDD), U1.14 (5V)
- new net C1: SW1.1, SW2.1, SW3.1
- new net C2: SW4.1, SW5.1, SW6.1
- new net C3: SW7.1, SW8.1, SW9.1
- new net GND: D12.3 (VSS), D13.3 (VSS), SW1.C, U1.13 (GND)
- new net R1: D1.1 (K), D4.1 (K), D7.1 (K)
- new net R2: D2.1 (K), D5.1 (K), D8.1 (K)
- new net R3: D3.1 (K), D6.1 (K), D9.1 (K)
